File: snowslide-pcb/snowslide-pcb.kicad_pcb (KiCad board)
At the start: 2 copper layers, 179.7 x 122.7 mm, 139 parts, among them J1 TRRS, J2 OLED, P1 i2c_pin, P2 i2c_pin, P3 battery+, P4 battery-, SW0 SW_Push, SW1 SW_Push, SW10 SW_Push, SW11 SW_Push, SW12 SW_Push, SW13 SW_Push, SW14 SW_Push, SW15 SW_Push, SW16 SW_Push, SW17 SW_Push, SW18 SW_Push, SW19 SW_Push, SW2 SW_Push, SW20 SW_Push, SW21 SW_Push, SW22 SW_Push, SW23 SW_Push, SW24 SW_Push, SW25 SW_Push, SW26 SW_Push, SW27 SW_Push, SW28 SW_Push, SW29 SW_Push, SW3 SW_Push, SW30 SW_Push, SW31 SW_Push, SW32 SW_Push, SW33 SW_DPDT_x2, SW34 SW_DPDT_x2, SW4 SW_Push, SW5 SW_Push, SW6 SW_Push, SW7 SW_Push, SW8 SW_Push, SW9 SW_Push, U1 ProMicro

Commit message: Added .gitignore
Parts:
- added J2: OLED, used_footprints:OLED_4Pin_SSD1306, F.Cu at (244.4, 121.3)
- added J2: OLED, used_footprints:OLED_4Pin_SSD1306, B.Cu at (165.6, 121.3)
- added L10: SK6812MINI_LED, used_footprints:YS-SK6812MINI-E, F.Cu at (156.9, 145.1)
- added L10: SK6812MINI_LED, used_footprints:YS-SK6812MINI-E, B.Cu at (253.1, 145.1)
- added L11: SK6812MINI_LED, used_footprints:YS-SK6812MINI-E, F.Cu at (139.1, 135.7)
- added L11: SK6812MINI_LED, used_footprints:YS-SK6812MINI-E, B.Cu at (270.9, 135.7)
- added L12: SK6812MINI_LED, used_footprints:YS-SK6812MINI-E, F.Cu at (139.1, 116.7)
- added L12: SK6812MINI_LED, used_footprints:YS-SK6812MINI-E, B.Cu at (270.9, 116.7)
- added L13: SK6812MINI_LED, used_footprints:YS-SK6812MINI-E, F.Cu at (139.1, 97.7)
- added L13: SK6812MINI_LED, used_footprints:YS-SK6812MINI-E, B.Cu at (270.9, 97.7)
- added L14: SK6812MINI_LED, used_footprints:YS-SK6812MINI-E, F.Cu at (139.1, 78.6)
- added L14: SK6812MINI_LED, used_footprints:YS-SK6812MINI-E, B.Cu at (270.9, 78.6)
- added L15: SK6812MINI_LED, used_footprints:YS-SK6812MINI-E, F.Cu at (120.0, 76.6)
- added L15: SK6812MINI_LED, used_footprints:YS-SK6812MINI-E, B.Cu at (290.0, 76.6)
- added L16: SK6812MINI_LED, used_footprints:YS-SK6812MINI-E, F.Cu at (120.0, 95.7)
- added L16: SK6812MINI_LED, used_footprints:YS-SK6812MINI-E, B.Cu at (290.0, 95.7)
- added L17: SK6812MINI_LED, used_footprints:YS-SK6812MINI-E, F.Cu at (120.0, 114.7)
- added L17: SK6812MINI_LED, used_footprints:YS-SK6812MINI-E, B.Cu at (290.0, 114.7)
- added L18: SK6812MINI_LED, used_footprints:YS-SK6812MINI-E, F.Cu at (120.0, 133.8)
- added L18: SK6812MINI_LED, used_footprints:YS-SK6812MINI-E, B.Cu at (290.0, 133.8)
- added L19: SK6812MINI_LED, used_footprints:YS-SK6812MINI-E, F.Cu at (131.7, 146.1)
- added L19: SK6812MINI_LED, used_footprints:YS-SK6812MINI-E, B.Cu at (278.3, 146.1)
- added L20: SK6812MINI_LED, used_footprints:YS-SK6812MINI-E, F.Cu at (109.6, 143.4)
- added L20: SK6812MINI_LED, used_footprints:YS-SK6812MINI-E, B.Cu at (300.4, 143.4)
- added L21: SK6812MINI_LED, used_footprints:YS-SK6812MINI-E, F.Cu at (101.0, 131.2)
- added L21: SK6812MINI_LED, used_footprints:YS-SK6812MINI-E, B.Cu at (309.0, 131.2)
- added L22: SK6812MINI_LED, used_footprints:YS-SK6812MINI-E, F.Cu at (101.0, 112.2)
- added L22: SK6812MINI_LED, used_footprints:YS-SK6812MINI-E, B.Cu at (309.0, 112.2)
- added L23: SK6812MINI_LED, used_footprints:YS-SK6812MINI-E, F.Cu at (100.9, 93.2)
- added L23: SK6812MINI_LED, used_footprints:YS-SK6812MINI-E, B.Cu at (309.1, 93.2)
- added L24: SK6812MINI_LED, used_footprints:YS-SK6812MINI-E, F.Cu at (101.0, 74.1)
- added L24: SK6812MINI_LED, used_footprints:YS-SK6812MINI-E, B.Cu at (309.0, 74.1)
- added L25: SK6812MINI_LED, used_footprints:YS-SK6812MINI-E, F.Cu at (81.9, 76.6)
- added L25: SK6812MINI_LED, used_footprints:YS-SK6812MINI-E, B.Cu at (328.1, 76.6)
- added L26: SK6812MINI_LED, used_footprints:YS-SK6812MINI-E, F.Cu at (81.9, 95.6)
- added L26: SK6812MINI_LED, used_footprints:YS-SK6812MINI-E, B.Cu at (328.1, 95.6)
- added L27: SK6812MINI_LED, used_footprints:YS-SK6812MINI-E, F.Cu at (81.9, 114.7)
- added L27: SK6812MINI_LED, used_footprints:YS-SK6812MINI-E, B.Cu at (328.1, 114.7)
- added L28: SK6812MINI_LED, used_footprints:YS-SK6812MINI-E, F.Cu at (81.9, 133.8)
- added L28: SK6812MINI_LED, used_footprints:YS-SK6812MINI-E, B.Cu at (328.1, 133.8)
- added L29: SK6812MINI_LED, used_footprints:YS-SK6812MINI-E, F.Cu at (87.8, 145.7)
- added L29: SK6812MINI_LED, used_footprints:YS-SK6812MINI-E, B.Cu at (322.2, 145.7)
- added L30: SK6812MINI_LED, used_footprints:YS-SK6812MINI-E, F.Cu at (62.8, 137.9)
- added L30: SK6812MINI_LED, used_footprints:YS-SK6812MINI-E, B.Cu at (347.2, 137.9)
- added L31: SK6812MINI_LED, used_footprints:YS-SK6812MINI-E, F.Cu at (61.8, 118.8)
- added L31: SK6812MINI_LED, used_footprints:YS-SK6812MINI-E, B.Cu at (348.2, 118.8)
- added L32: SK6812MINI_LED, used_footprints:YS-SK6812MINI-E, F.Cu at (60.8, 99.8)
- added L32: SK6812MINI_LED, used_footprints:YS-SK6812MINI-E, B.Cu at (349.2, 99.8)
- added L33: SK6812MINI_LED, used_footprints:YS-SK6812MINI-E, F.Cu at (59.8, 80.8)
- added L33: SK6812MINI_LED, used_footprints:YS-SK6812MINI-E, B.Cu at (350.2, 80.8)
- added L34: SK6812MINI_LED, used_footprints:YS-SK6812MINI-E, F.Cu at (40.8, 81.8)
- added L34: SK6812MINI_LED, used_footprints:YS-SK6812MINI-E, B.Cu at (369.2, 81.8)
- added L35: SK6812MINI_LED, used_footprints:YS-SK6812MINI-E, F.Cu at (41.8, 100.8)
- added L35: SK6812MINI_LED, used_footprints:YS-SK6812MINI-E, B.Cu at (368.2, 100.8)
- added L36: SK6812MINI_LED, used_footprints:YS-SK6812MINI-E, F.Cu at (42.8, 119.8)
- added L36: SK6812MINI_LED, used_footprints:YS-SK6812MINI-E, B.Cu at (367.2, 119.8)
- added L37: SK6812MINI_LED, used_footprints:YS-SK6812MINI-E, F.Cu at (43.8, 138.9)
- added L37: SK6812MINI_LED, used_footprints:YS-SK6812MINI-E, B.Cu at (366.2, 138.9)
- added L38: SK6812MINI_LED, used_footprints:YS-SK6812MINI-E, F.Cu at (23.9, 123.1)
- added L38: SK6812MINI_LED, used_footprints:YS-SK6812MINI-E, B.Cu at (386.1, 123.1)
- added L7: SK6812MINI_LED, used_footprints:YS-SK6812MINI-E, F.Cu at (152.6, 153.8)
- added L7: SK6812MINI_LED, used_footprints:YS-SK6812MINI-E, B.Cu at (257.4, 153.8)
- added L8: SK6812MINI_LED, used_footprints:YS-SK6812MINI-E, F.Cu at (171.1, 166.1)
- added L8: SK6812MINI_LED, used_footprints:YS-SK6812MINI-E, B.Cu at (238.9, 166.1)
- added L9: SK6812MINI_LED, used_footprints:YS-SK6812MINI-E, F.Cu at (177.3, 158.8)
- added L9: SK6812MINI_LED, used_footprints:YS-SK6812MINI-E, B.Cu at (232.7, 158.8)
- added SW0: SW_Push, used_footprints:Switch_Reset_THT, F.Cu at (177.6, 97.5)
- added SW0: SW_Push, used_footprints:Switch_Reset_THT, B.Cu at (232.4, 97.5)
- added SW1: SW_Push, used_footprints:CherryMX_MidHeight_Hotswap_1u, F.Cu at (40.5, 77.1)
- added SW1: SW_Push, used_footprints:CherryMX_MidHeight_Hotswap_1u, B.Cu at (369.5, 77.1)
- added SW10: SW_Push, used_footprints:CherryMX_MidHeight_Hotswap_1u, F.Cu at (101.0, 88.5)
- added SW10: SW_Push, used_footprints:CherryMX_MidHeight_Hotswap_1u, B.Cu at (309.0, 88.5)
- added SW11: SW_Push, used_footprints:CherryMX_MidHeight_Hotswap_1u, F.Cu at (120.0, 91.0)
- added SW11: SW_Push, used_footprints:CherryMX_MidHeight_Hotswap_1u, B.Cu at (290.0, 91.0)
- added SW12: SW_Push, used_footprints:CherryMX_MidHeight_Hotswap_1u, F.Cu at (139.1, 92.9)
- added SW12: SW_Push, used_footprints:CherryMX_MidHeight_Hotswap_1u, B.Cu at (270.9, 92.9)
- added SW13: SW_Push, used_footprints:CherryMX_MidHeight_Hotswap_1u, F.Cu at (42.5, 115.1)
- added SW13: SW_Push, used_footprints:CherryMX_MidHeight_Hotswap_1u, B.Cu at (367.5, 115.1)
- added SW14: SW_Push, used_footprints:CherryMX_MidHeight_Hotswap_1u, F.Cu at (61.6, 114.1)
- added SW14: SW_Push, used_footprints:CherryMX_MidHeight_Hotswap_1u, B.Cu at (348.4, 114.1)
- added SW15: SW_Push, used_footprints:CherryMX_MidHeight_Hotswap_1u, F.Cu at (81.9, 110.0)
- added SW15: SW_Push, used_footprints:CherryMX_MidHeight_Hotswap_1u, B.Cu at (328.1, 110.0)
- added SW16: SW_Push, used_footprints:CherryMX_MidHeight_Hotswap_1u, F.Cu at (100.9, 107.5)
- added SW16: SW_Push, used_footprints:CherryMX_MidHeight_Hotswap_1u, B.Cu at (309.1, 107.5)
- added SW17: SW_Push, used_footprints:CherryMX_MidHeight_Hotswap_1u, F.Cu at (120.0, 110.0)
- added SW17: SW_Push, used_footprints:CherryMX_MidHeight_Hotswap_1u, B.Cu at (290.0, 110.0)
- added SW18: SW_Push, used_footprints:CherryMX_MidHeight_Hotswap_1u, F.Cu at (139.1, 112.0)
- added SW18: SW_Push, used_footprints:CherryMX_MidHeight_Hotswap_1u, B.Cu at (270.9, 112.0)
- added SW19: SW_Push, used_footprints:CherryMX_MidHeight_Hotswap_1u, F.Cu at (180.4, 155.2)
- added SW19: SW_Push, used_footprints:CherryMX_MidHeight_Hotswap_1u, B.Cu at (229.6, 155.2)
- added SW2: SW_Push, used_footprints:CherryMX_MidHeight_Hotswap_1u, F.Cu at (59.6, 76.1)
- added SW2: SW_Push, used_footprints:CherryMX_MidHeight_Hotswap_1u, B.Cu at (350.4, 76.1)
- added SW20: SW_Push, used_footprints:CherryMX_MidHeight_Hotswap_1u, F.Cu at (43.5, 134.2)
- added SW20: SW_Push, used_footprints:CherryMX_MidHeight_Hotswap_1u, B.Cu at (366.5, 134.2)
- added SW21: SW_Push, used_footprints:CherryMX_MidHeight_Hotswap_1u, F.Cu at (62.6, 133.2)
- added SW21: SW_Push, used_footprints:CherryMX_MidHeight_Hotswap_1u, B.Cu at (347.4, 133.2)
- added SW22: SW_Push, used_footprints:CherryMX_MidHeight_Hotswap_1u, F.Cu at (81.9, 129.1)
- added SW22: SW_Push, used_footprints:CherryMX_MidHeight_Hotswap_1u, B.Cu at (328.1, 129.1)
- added SW23: SW_Push, used_footprints:CherryMX_MidHeight_Hotswap_1u, F.Cu at (101.0, 126.5)
- added SW23: SW_Push, used_footprints:CherryMX_MidHeight_Hotswap_1u, B.Cu at (309.0, 126.5)
- added SW24: SW_Push, used_footprints:CherryMX_MidHeight_Hotswap_1u, F.Cu at (120.0, 129.1)
- added SW24: SW_Push, used_footprints:CherryMX_MidHeight_Hotswap_1u, B.Cu at (290.0, 129.1)
- added SW25: SW_Push, used_footprints:CherryMX_MidHeight_Hotswap_1u, F.Cu at (139.1, 131.1)
- added SW25: SW_Push, used_footprints:CherryMX_MidHeight_Hotswap_1u, B.Cu at (270.9, 131.1)
- added SW26: SW_Push, used_footprints:CherryMX_MidHeight_Hotswap_1u, F.Cu at (159.1, 141.0)
- added SW26: SW_Push, used_footprints:CherryMX_MidHeight_Hotswap_1u, B.Cu at (250.9, 141.0)
- added SW27: SW_Push, used_footprints:CherryMX_MidHeight_Hotswap_1u, F.Cu at (23.6, 118.4)
- added SW27: SW_Push, used_footprints:CherryMX_MidHeight_Hotswap_1u, B.Cu at (386.4, 118.4)
- added SW28: SW_Push, used_footprints:CherryMX_MidHeight_Hotswap_1u, F.Cu at (88.8, 150.3)
- added SW28: SW_Push, used_footprints:CherryMX_MidHeight_Hotswap_1u, B.Cu at (321.2, 150.3)
- added SW29: SW_Push, used_footprints:CherryMX_MidHeight_Hotswap_1u, F.Cu at (109.6, 148.1)
- added SW29: SW_Push, used_footprints:CherryMX_MidHeight_Hotswap_1u, B.Cu at (300.4, 148.1)
- added SW3: SW_Push, used_footprints:CherryMX_MidHeight_Hotswap_1u, F.Cu at (81.9, 71.9)
- added SW3: SW_Push, used_footprints:CherryMX_MidHeight_Hotswap_1u, B.Cu at (328.1, 71.9)
- added SW30: SW_Push, used_footprints:CherryMX_MidHeight_Hotswap_1u, F.Cu at (130.6, 150.6)
- added SW30: SW_Push, used_footprints:CherryMX_MidHeight_Hotswap_1u, B.Cu at (279.4, 150.6)
- added SW31: SW_Push, used_footprints:CherryMX_MidHeight_Hotswap_1u, F.Cu at (150.4, 157.9)
- added SW31: SW_Push, used_footprints:CherryMX_MidHeight_Hotswap_1u, B.Cu at (259.6, 157.9)
- added SW32: SW_Push, used_footprints:CherryMX_MidHeight_Hotswap_1u, F.Cu at (168.0, 169.7)
- added SW32: SW_Push, used_footprints:CherryMX_MidHeight_Hotswap_1u, B.Cu at (242.0, 169.7)
- added SW4: SW_Push, used_footprints:CherryMX_MidHeight_Hotswap_1u, F.Cu at (100.9, 69.4)
- added SW4: SW_Push, used_footprints:CherryMX_MidHeight_Hotswap_1u, B.Cu at (309.1, 69.4)
- added SW5: SW_Push, used_footprints:CherryMX_MidHeight_Hotswap_1u, F.Cu at (120.0, 71.9)
- added SW5: SW_Push, used_footprints:CherryMX_MidHeight_Hotswap_1u, B.Cu at (290.0, 71.9)
- added SW6: SW_Push, used_footprints:CherryMX_MidHeight_Hotswap_1u, F.Cu at (139.1, 73.9)
- added SW6: SW_Push, used_footprints:CherryMX_MidHeight_Hotswap_1u, B.Cu at (270.9, 73.9)
- added SW7: SW_Push, used_footprints:CherryMX_MidHeight_Hotswap_1u, F.Cu at (41.5, 96.1)
- added SW7: SW_Push, used_footprints:CherryMX_MidHeight_Hotswap_1u, B.Cu at (368.5, 96.1)
- added SW8: SW_Push, used_footprints:CherryMX_MidHeight_Hotswap_1u, F.Cu at (60.6, 95.1)
- added SW8: SW_Push, used_footprints:CherryMX_MidHeight_Hotswap_1u, B.Cu at (349.4, 95.1)
- added SW9: SW_Push, used_footprints:CherryMX_MidHeight_Hotswap_1u, F.Cu at (81.9, 91.0)
- added SW9: SW_Push, used_footprints:CherryMX_MidHeight_Hotswap_1u, B.Cu at (328.1, 91.0)
Other:
- board size 179.7 x 122.7 mm -> 633.7 x 197.6 mm

Commit message: PCB layout completed.
Parts:
- removed D1, D10, D11, D12, D13, D14, D15, D16, D17, D18, D19, D2, D20, D21, D22, D23, D24, D25, D26, D27, D28, D29, D3, D30, D31, D32, D4, D5, D6, D7, D8, D9: 1N4148, used_footprints:diode_TH_SMD
- removed ENC1, ENC2, ENC3: Rotary_Encoder_Switch, used_footprints:RotaryEncoder_Alps_EC11E-Switch_Vertical_H20mm-keebio_modified
- removed H15: MountingHole, used_footprints:M2_HOLE_PCB
- removed HM1, HM10, HM11, HM12, HM13, HM14, HM2, HM3, HM4, HM5, HM6, HM7, HM8, HM9: CaseHole, used_footprints:M2_HOLE_PCB
- removed J1: TRRS, used_footprints:MJ-4PP-9
- removed the J2 at (244.4, 121.3)
- removed the J2 at (-85.6, 46.4)
- removed JP1, JP12, JP2, JP3, JP4, JP5, JP6, JP7, JP8: Device_Jumper_NO_Small, used_footprints:avalanche_Jumper
- removed JP10, JP11, JP9: Device_Jumper_NO_Small, used_footprints:Jumper_rev
- removed L10 (x3), L11 (x3), L12 (x3), L13 (x3), L14 (x3), L15 (x3), L16 (x3), L17 (x3), L18 (x3), L19 (x3), L20 (x3), L21 (x3), L22 (x3), L23 (x3), L24 (x3), L25 (x3), L26 (x3), L27 (x3), L28 (x3), L29 (x3), L30 (x3), L31 (x3), L32 (x3), L33 (x3), L34 (x3), L35 (x3), L36 (x3), L37 (x3), L38 (x3), L7 (x3), L8 (x3), L9 (x3): SK6812MINI_LED, used_footprints:YS-SK6812MINI-E
- removed P1, P2: i2c_pin, used_footprints:1pin_conn
- removed P3: battery+, used_footprints:1pin_conn
- removed P4: battery-, used_footprints:1pin_conn
- removed R1, R2: 4.7K, used_footprints:Resistor_Hybrid_1205
- removed SW0 (x3): SW_Push, used_footprints:Switch_Reset_THT
- removed SW1 (x3), SW10 (x3), SW11 (x3), SW12 (x3), SW13 (x3), SW14 (x3), SW15 (x3), SW16 (x3), SW17 (x3), SW18 (x3), SW19 (x3), SW2 (x3), SW20 (x3), SW21 (x3), SW22 (x3), SW23 (x3), SW24 (x3), SW25 (x3), SW26 (x3), SW27 (x3), SW28 (x3), SW29 (x3), SW3 (x3), SW30 (x3), SW31 (x3), SW32 (x3), SW4 (x3), SW5 (x3), SW6 (x3), SW7 (x3), SW8 (x3), SW9 (x3): SW_Push, used_footprints:CherryMX_MidHeight_Hotswap_1u
- removed SW33, SW34: SW_DPDT_x2, used_footprints:Switch_MSK-12C01-07
- removed U1: ProMicro, used_footprints:ProMicro_rev2
- removed W1: jumper, used_footprints:avalanche_Jumper
- moved J2 42.3 mm to (205.0, 136.5)
Routing:
- net (no net): track 8043.1 -> 0.00 mm, vias 391 -> 0
Other:
- board size 633.7 x 197.6 mm -> 69.5 x 58.5 mm
- board text removed: "Avalanche v4.2 designed by vitvlkv"
- board text removed: "W1"
- board text removed: "https://github.com/vlkv/avalanche"
